Commit message: update file pathes in some launch files.
Signed-off-by: ShoTakahashi <takahashi@techno-road.com>

File: src/kobuki_description/urdf/kobuki.urdf.xacro (robot description, xacro)
@@ -7,6 +7,6 @@
  -->
 <robot name="kobuki" xmlns:xacro="http://ros.org/wiki/xacro">
-  <xacro:include filename="/home/takahashi/turtlebot_ws/src/kobuki_description/urdf/common_properties.urdf.xacro"/>
-  <xacro:include filename="/home/takahashi/turtlebot_ws/src/kobuki_description/urdf/kobuki_gazebo.urdf.xacro"/>
+  <xacro:include filename="$(find kobuki_description)/urdf/common_properties.urdf.xacro"/>
+  <xacro:include filename="$(find kobuki_description)/urdf/kobuki_gazebo.urdf.xacro"/>
   <xacro:property name="wheel_sep" value="0.23" />
    <!-- Kobuki -->

File: src/kobuki_description/urdf/kobuki_gazebo.urdf.xacro (robot description, xacro)
@@ -38,6 +38,5 @@
 	  </gazebo>
 	  <gazebo>
-	    <plugin name="kobuki_controller" filename="/home/takahashi/turtlebot_ws/devel/lib/libgazebo_ros_kobuki.so">
-<!--	    <plugin name="kobuki_controller" filename="libgazebo_ros_kobuki.so">-->
+	    <plugin name="kobuki_controller" filename="libgazebo_ros_kobuki.so">
 	      <publish_tf>1</publish_tf>
 	      <left_wheel_joint_name>wheel_left_joint</left_wheel_joint_name>

File: src/turtlebot/turtlebot_description/robots/kobuki_hexagons_kinect.urdf.xacro (robot description, xacro)
@@ -6,5 +6,5 @@
 -->
 <robot name="turtlebot" xmlns:xacro="http://ros.org/wiki/xacro">
-  <xacro:include filename="/home/takahashi/turtlebot_ws/src/turtlebot/turtlebot_description/urdf/turtlebot_library.urdf.xacro" />
+  <xacro:include filename="$(find turtlebot_description)/urdf/turtlebot_library.urdf.xacro" />
   <kobuki/>
   <stack_hexagons parent="base_link"/>

File: src/turtlebot/turtlebot_description/urdf/sensors/kinect.urdf.xacro (robot description, xacro)
@@ -1,6 +1,6 @@
 <?xml version="1.0"?>
 <robot name="sensor_kinect" xmlns:xacro="http://ros.org/wiki/xacro">
-  <xacro:include filename="/home/takahashi/turtlebot_ws/src/turtlebot/turtlebot_description/urdf/turtlebot_gazebo.urdf.xacro"/>
-  <xacro:include filename="/home/takahashi/turtlebot_ws/src/turtlebot/turtlebot_description/urdf/turtlebot_properties.urdf.xacro"/>
+  <xacro:include filename="$(find turtlebot_description)/urdf/turtlebot_gazebo.urdf.xacro"/>
+  <xacro:include filename="$(find turtlebot_description)/urdf/turtlebot_properties.urdf.xacro"/>
   <xacro:property name="kinect_cam_py" value="-0.0125"/>
   <!-- Parameterised in part by the values in turtlebot_properties.urdf.xacro -->
@@ -12,5 +12,6 @@
       <limit effort="1000.0" lower="-0.521567881107" upper="0.521567881107" velocity="10"/>
 <!--      <limit effort="1000.0" lower="-1.57" upper="1.57" velocity="10"/>-->
-      <origin xyz="0.07 ${kinect_cam_py} ${cam_pz}" rpy="${cam_or} ${cam_op} ${cam_oy}"/>
+      <origin xyz="0.07 0.0 0.11" rpy="${cam_or} ${cam_op} ${cam_oy}"/>
+<!-- 0614     <origin xyz="0.07 ${kinect_cam_py} ${cam_pz}" rpy="${cam_or} ${cam_op} ${cam_oy}"/>-->
 <!--      <origin xyz="${cam_px} ${kinect_cam_py} ${cam_pz}" rpy="${cam_or} ${cam_op} ${cam_oy}"/>-->
       <parent link="${parent}"/>
@@ -25,5 +26,6 @@
     <link name="camera_rgb_optical_frame"/>
     <joint name="camera_joint" type="fixed">
-      <origin xyz="-0.0 ${-kinect_cam_py} -0.016" rpy="0 0 0"/>
+      <origin xyz="0.0 0.0 -0.016" rpy="0 0 0"/>
+<!--      <origin xyz="-0.0 ${-kinect_cam_py} -0.016" rpy="0 0 0"/>-->
       <parent link="camera_rgb_frame"/>
       <child link="camera_link"/>
@@ -40,13 +42,14 @@
        <origin xyz="0 0 0" rpy="0 0 ${M_PI/2}"/>
         <geometry>
-         <mesh filename="package://turtlebot_description/meshes/sensors/kinect.dae"/>
+<!--         <mesh filename="package://turtlebot_description/meshes/sensors/kinect.dae"/>-->
+  	      <box size="0.01 0.02 0.04"/>
         </geometry>
       </visual>
-  	  <collision>
-        <origin xyz="0.0 0.0 0.0" rpy="0 0 0"/>
-  	    <geometry>
-  	      <box size="0.07271 0.27794 0.073"/>
-  	    </geometry>
-  	  </collision>
+<!--  	  <collision>-->
+<!--        <origin xyz="0.0 0.0 0.0" rpy="0 0 0"/>-->
+<!--  	    <geometry>-->
+<!--  	      <box size="0.01 0.02 0.04"/>-->
+<!--  	    </geometry>-->
+<!--  	  </collision>-->
       <inertial>
         <mass value="0.564" />

File: src/turtlebot/turtlebot_description/urdf/stacks/hexagons.urdf.xacro (robot description, xacro)
@@ -16,16 +16,16 @@
     </joint>
     <link name="pole_bottom_${number}_link">
-      <visual>
-        <origin xyz="0 0 0" rpy="0 0 0"/>
-        <geometry>
-          <mesh filename="package://turtlebot_description/meshes/stacks/hexagons/pole_bottom.dae"/>
-        </geometry>
-      </visual>
-      <collision>
-        <origin xyz="0 0 0" rpy="0 0 0"/>
-        <geometry>
-          <cylinder length="0.0492" radius="0.006"/>
-        </geometry>
-      </collision>
+<!--      <visual>-->
+<!--        <origin xyz="0 0 0" rpy="0 0 0"/>-->
+<!--        <geometry>-->
+<!--          <mesh filename="package://turtlebot_description/meshes/stacks/hexagons/pole_bottom.dae"/>-->
+<!--        </geometry>-->
+<!--      </visual>-->
+<!--      <collision>-->
+<!--        <origin xyz="0 0 0" rpy="0 0 0"/>-->
+<!--        <geometry>-->
+<!--          <cylinder length="0.0492" radius="0.006"/>-->
+<!--        </geometry>-->
+<!--      </collision>-->
       <inertial>
         <mass value="0.008"/>
@@ -44,16 +44,16 @@
     </joint>
     <link name="pole_middle_${number}_link">
-      <visual>
-        <origin xyz="0 0 0" rpy="0 ${M_PI} 0"/>
-        <geometry>
-          <mesh filename="package://turtlebot_description/meshes/stacks/hexagons/pole_middle.dae"/>
-        </geometry>
-      </visual>
-      <collision>
-        <origin xyz="0 0 0" rpy="0 0 0"/>
-        <geometry>
-          <cylinder length="0.0608" radius="0.006"/>
-        </geometry>
-      </collision>
+<!--      <visual>-->
+<!--        <origin xyz="0 0 0" rpy="0 ${M_PI} 0"/>-->
+<!--        <geometry>-->
+<!--          <mesh filename="package://turtlebot_description/meshes/stacks/hexagons/pole_middle.dae"/>-->
+<!--        </geometry>-->
+<!--      </visual>-->
+<!--      <collision>-->
+<!--        <origin xyz="0 0 0" rpy="0 0 0"/>-->
+<!--        <geometry>-->
+<!--          <cylinder length="0.0608" radius="0.006"/>-->
+<!--        </geometry>-->
+<!--      </collision>-->
       <inertial>
         <mass value="0.012"/>
@@ -72,16 +72,16 @@
     </joint>
     <link name="pole_top_${number}_link">
-      <visual>
-        <origin xyz=" 0 0 0" rpy="0 0 0"/>
-        <geometry>
-          <mesh filename="package://turtlebot_description/meshes/stacks/hexagons/pole_top.dae"/>
-        </geometry>
-      </visual>
-      <collision>
-        <origin xyz="0 0 0" rpy="0 0 0"/>
-        <geometry>
-          <cylinder length="0.2032" radius="0.006"/>
-        </geometry>
-      </collision>
+<!--      <visual>-->
+<!--        <origin xyz=" 0 0 0" rpy="0 0 0"/>-->
+<!--        <geometry>-->
+<!--          <mesh filename="package://turtlebot_description/meshes/stacks/hexagons/pole_top.dae"/>-->
+<!--        </geometry>-->
+<!--      </visual>-->
+<!--      <collision>-->
+<!--        <origin xyz="0 0 0" rpy="0 0 0"/>-->
+<!--        <geometry>-->
+<!--          <cylinder length="0.2032" radius="0.006"/>-->
+<!--        </geometry>-->
+<!--      </collision>-->
       <inertial>
         <mass value="0.060"/>
@@ -100,16 +100,16 @@
     </joint>
     <link name="pole_kinect_${number}_link">
-      <visual>
-        <origin xyz="0 0 -0.01" rpy="0 0 0"/>
-        <geometry>
-          <mesh filename="package://turtlebot_description/meshes/sensors/sensor_pole.dae" />
-        </geometry>
-      </visual>
-      <collision>
-        <origin xyz="0 0 0" rpy="0 0 0"/>
-        <geometry>
-          <cylinder length="0.0936" radius="0.006"/>
-        </geometry>
-      </collision>
+<!--      <visual>-->
+<!--        <origin xyz="0 0 -0.01" rpy="0 0 0"/>-->
+<!--        <geometry>-->
+<!--          <mesh filename="package://turtlebot_description/meshes/sensors/sensor_pole.dae" />-->
+<!--        </geometry>-->
+<!--      </visual>-->
+<!--      <collision>-->
+<!--        <origin xyz="0 0 0" rpy="0 0 0"/>-->
+<!--        <geometry>-->
+<!--          <cylinder length="0.0936" radius="0.006"/>-->
+<!--        </geometry>-->
+<!--      </collision>-->
       <inertial>
         <mass value="0.020"/>
@@ -139,16 +139,16 @@
     </joint>
     <link name="plate_bottom_link">
-      <visual>
-        <origin xyz="0 0 0" rpy="0 0 0"/>
-        <geometry>
-          <mesh filename="package://turtlebot_description/meshes/stacks/hexagons/plate_bottom.dae"/>
-        </geometry>
-      </visual>
-      <collision>
-        <origin xyz="-0.02364 0 0" rpy="0 0 0"/>
-        <geometry>
-          <cylinder length="0.006" radius="0.170"/>
-        </geometry>
-      </collision>
+<!--      <visual>-->
+<!--        <origin xyz="0 0 0" rpy="0 0 0"/>-->
+<!--        <geometry>-->
+<!--          <mesh filename="package://turtlebot_description/meshes/stacks/hexagons/plate_bottom.dae"/>-->
+<!--        </geometry>-->
+<!--      </visual>  -->
+<!--      <collision>-->
+<!--        <origin xyz="-0.02364 0 0" rpy="0 0 0"/>-->
+<!--        <geometry>-->
+<!--          <cylinder length="0.006" radius="0.170"/>-->
+<!--        </geometry>-->
+<!--      </collision>-->
       <inertial>
         <mass value="0.520" />
@@ -169,16 +169,16 @@
     </joint>
     <link name="plate_middle_link">
-      <visual>
-        <origin xyz="0 0 0" rpy="0 0 0"/>
-        <geometry>
-          <mesh filename="package://turtlebot_description/meshes/stacks/hexagons/plate_middle.dae"/>
-        </geometry>
-      </visual>
-      <collision>
-        <origin xyz="0.01364 0.0 0.0" rpy="0 0 0"/>
-        <geometry>
-          <cylinder length="0.006" radius="0.170"/>
-        </geometry>
-      </collision>
+<!--      <visual>-->
+<!--        <origin xyz="0 0 0" rpy="0 0 0"/>-->
+<!--        <geometry>-->
+<!--          <mesh filename="package://turtlebot_description/meshes/stacks/hexagons/plate_middle.dae"/>-->
+<!--        </geometry>-->
+<!--      </visual>  -->
+<!--      <collision>-->
+<!--        <origin xyz="0.01364 0.0 0.0" rpy="0 0 0"/>-->
+<!--        <geometry>-->
+<!--          <cylinder length="0.006" radius="0.170"/>-->
+<!--        </geometry>-->
+<!--      </collision>-->
       <inertial>
         <mass value="0.520" />
@@ -201,16 +201,16 @@
     </joint>
     <link name="plate_top_link">
-      <visual>
-        <origin xyz="0 0 0" rpy="0 0 0"/>
-        <geometry>
-          <mesh filename="package://turtlebot_description/meshes/stacks/hexagons/plate_top.dae"/>
-        </geometry>
-      </visual>
-      <collision>
-        <origin xyz="0.01364 0 0" rpy="0 0 0"/>
-        <geometry>
-          <cylinder length="0.006" radius="0.170"/>
-        </geometry>
-      </collision>
+<!--      <visual>-->
+<!--        <origin xyz="0 0 0" rpy="0 0 0"/>-->
+<!--        <geometry>-->
+<!--          <mesh filename="package://turtlebot_description/meshes/stacks/hexagons/plate_top.dae"/>-->
+<!--        </geometry>-->
+<!--      </visual>  -->
+<!--      <collision>-->
+<!--        <origin xyz="0.01364 0 0" rpy="0 0 0"/>-->
+<!--        <geometry>-->
+<!--          <cylinder length="0.006" radius="0.170"/>-->
+<!--        </geometry>-->
+<!--      </collision>-->
       <inertial>
         <mass value="0.520"/>

File: src/turtlebot/turtlebot_description/urdf/turtlebot_gazebo.urdf.xacro (robot description, xacro)
@@ -80,5 +80,5 @@
         </noise>
       </ray>
-      <plugin name="gazebo_ros_head_hokuyo_controller" filename="/home/takahashi/turtlebot_ws/devel/lib/libgazebo_ros_gpu_laser.so">
+      <plugin name="gazebo_ros_head_hokuyo_controller" filename="libgazebo_ros_gpu_laser.so">
         <topicName>scan2</topicName>
         <frameName>camera_depth_frame</frameName>
@@ -87,5 +87,5 @@
   </gazebo>
   <gazebo>
-      <plugin name="gazebo_ros_head_hokuyo_controller" filename="/home/takahashi/turtlebot_ws/devel/lib/libgazebo_ros_template.so">
+      <plugin name="gazebo_ros_head_hokuyo_controller" filename="libgazebo_ros_template.so">
       </plugin>
   </gazebo>

File: src/turtlebot/turtlebot_description/urdf/turtlebot_library.urdf.xacro (robot description, xacro)
@@ -5,16 +5,15 @@
 <robot xmlns:xacro="http://ros.org/wiki/xacro">
   <!-- General -->
-  <xacro:include filename="/home/takahashi/turtlebot_ws/src/turtlebot/turtlebot_description/urdf/common_properties.urdf.xacro"/>
-  <xacro:include filename="/home/takahashi/turtlebot_ws/src/turtlebot/turtlebot_description/urdf/turtlebot_properties.urdf.xacro"/>
+  <xacro:include filename="$(find turtlebot_description)/urdf/common_properties.urdf.xacro"/>
+  <xacro:include filename="$(find turtlebot_description)/urdf/turtlebot_properties.urdf.xacro"/>
   <!-- Bases -->
   <xacro:include filename="$(find create_description)/urdf/create.urdf.xacro"/>
-<xacro:include filename="/home/takahashi/turtlebot_ws/src/kobuki_description/urdf/kobuki.urdf.xacro" />
-<!--<xacro:include filename="$(find kobuki_description)/urdf/kobuki.urdf.xacro" />-->
+  <xacro:include filename="$(find kobuki_description)/urdf/kobuki.urdf.xacro" />
   <!-- Stacks -->
-  <xacro:include filename="/home/takahashi/turtlebot_ws/src/turtlebot/turtlebot_description/urdf/stacks/circles.urdf.xacro"/>
-  <xacro:include filename="/home/takahashi/turtlebot_ws/src/turtlebot/turtlebot_description/urdf/stacks/hexagons.urdf.xacro"/>
+  <xacro:include filename="$(find turtlebot_description)/urdf/stacks/circles.urdf.xacro"/>
+  <xacro:include filename="$(find turtlebot_description)/urdf/stacks/hexagons.urdf.xacro"/>
   <!-- 3D Sensors -->
-  <xacro:include filename="/home/takahashi/turtlebot_ws/src/turtlebot/turtlebot_description/urdf/sensors/kinect.urdf.xacro"/>
-  <xacro:include filename="/home/takahashi/turtlebot_ws/src/turtlebot/turtlebot_description/urdf/sensors/asus_xtion_pro.urdf.xacro"/>
-  <xacro:include filename="/home/takahashi/turtlebot_ws/src/turtlebot/turtlebot_description/urdf/sensors/asus_xtion_pro_offset.urdf.xacro"/>
+  <xacro:include filename="$(find turtlebot_description)/urdf/sensors/kinect.urdf.xacro"/>
+  <xacro:include filename="$(find turtlebot_description)/urdf/sensors/asus_xtion_pro.urdf.xacro"/>
+  <xacro:include filename="$(find turtlebot_description)/urdf/sensors/asus_xtion_pro_offset.urdf.xacro"/>
 </robot>
